File: zigtherm.brd (EAGLE design)
At the start: 27.6 x 26.7 mm, 22 parts, among them IC1 ATSAMR21E, IC2 TPS73033DBV, X1 USB-MICRO-B-BOTTOM-MOLEX

Commit message: XXX
Parts:
- added C12: 10n, rcl:C0603
- added JP5, JP6, JP7: PINH1X01SMD, pinhead_smd:PINH1X01SMD
- added R1: 0, rcl:R0603
- C1, C11, C2, C6, C7, C9: device rcl:C0402K -> rcl:C0603
- moved JP1 5.08 mm to (0.00, 12.7)
- moved X1 3.17 mm to (0.00, 21.0)
- moved C7 2.84 mm to (10.2, 19.1), flipped to the bottom, turned to 0 degrees
- moved IC2 2.54 mm to (10.2, 21.6), flipped to the bottom, turned to 90 degrees
- moved JP2 2.54 mm to (0.00, 5.08)
- moved JP3 2.54 mm to (0.00, 7.62)
- moved JP4 2.54 mm to (0.00, 7.62)
- moved C6 2.31 mm to (7.30, 21.6), flipped to the bottom, turned to 270 degrees
- moved C9 1.24 mm to (6.03, 15.4)
- moved C2 0.81 mm to (11.6, 18.9)
- moved C11 0.71 mm to (9.21, 19.1), flipped to the top, turned to 90 degrees
- moved C1 0.22 mm to (7.46, 15.4), flipped to the bottom
Connections:
- new net N$2: C12.1, IC2.4
- new net RST_N: IC1.26, JP5.1
- new net RX: IC1.27, JP6.1
- new net TX: IC1.25, JP7.1
- net AGND: now also R1.2
- net GND: now also C12.2, R1.1
Routing:
- net GND: track 23.9 -> 36.6 mm
- net TX: track 0.00 -> 11.0 mm, vias 0 -> 1
- net RX: track 0.00 -> 9.44 mm
- net RST_N: track 0.00 -> 7.85 mm
- net VDD: track 26.8 -> 22.8 mm, vias 3 -> 2
- net USB_DM: track 8.81 -> 12.0 mm
- net USB_DP: track 7.66 -> 10.8 mm
- net SWDIO: track 9.46 -> 12.0 mm
- net SWCLK: track 7.87 -> 10.0 mm
- net N$2: track 0.00 -> 2.04 mm
- net DVDD: track 1.23 -> 1.84 mm
- net VDDCORE: track 2.33 -> 2.71 mm, vias 0 -> 1
- net VBUS: track 9.47 -> 9.65 mm, vias 0 -> 1
- removed copper zone on layer 1, net AGND
- removed copper zone on layer 16, net GND
Other:
- board size 27.6 x 26.7 mm -> 27 x 26.7 mm

Commit message: Final design.
Parts:
- C10, C4, C5, C8: device rcl:C0402K -> rcl:C0603
- C3: device rcl:C0402 -> rcl:C0603
- moved L1 8.54 mm to (15.9, 17.1), turned to 270 degrees
- moved JP1 5.08 mm to (0.00, 7.62)
- moved C9 4.46 mm to (10.5, 15.1)
- moved C10 4.02 mm to (14.6, 6.99)
- moved C8 4.02 mm to (13.3, 6.99)
- moved C3 3.24 mm to (15.9, 6.99), turned to 270 degrees
- moved C5 3.18 mm to (7.62, 6.35)
- moved R1 2.71 mm to (14.9, 24.1)
- moved C4 2.69 mm to (10.2, 4.45)
- moved JP3 2.54 mm to (0.00, 5.08), flipped to the bottom, turned to 270 degrees
- moved AE1 2.54 mm to (21.6, 15.2)
- moved JP5 2.54 mm to (0.00, 10.2), flipped to the bottom, turned to 270 degrees
- moved JP6 2.54 mm to (0.00, 12.7)
- moved JP7 2.54 mm to (0.00, 12.7)
- moved X2 2.29 mm to (10.2, 7.62)
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Routing:
- net AGND: track 0.00 -> 74.4 mm, vias 0 -> 31
- net GND: track 36.6 -> 83.1 mm, vias 3 -> 13
- net VDD: track 22.8 -> 31.5 mm
- net VDDANA: track 6.00 -> 13.4 mm
- net RST_N: track 7.85 -> 12.5 mm, vias 0 -> 1
- net VDDCORE: track 2.71 -> 6.86 mm
- net N$3: track 5.77 -> 9.29 mm
- net SWCLK: track 10.0 -> 12.4 mm, vias 0 -> 1
- net N$7: track 4.83 -> 7.14 mm
- net USB_DP: track 10.8 -> 12.7 mm
- net USB_DM: track 12.0 -> 13.9 mm
- net VBUS: track 9.65 -> 11.6 mm
- net N$2: track 2.04 -> 2.68 mm
- net N$1: track 3.42 -> 4.05 mm
- net AVDD: track 4.40 -> 4.96 mm
- added copper zone on layer 1, net AGND
- added copper zone on layer 16, net AGND
- added copper zone on layer 1, net GND
- added copper zone on layer 16, net GND
Other:
- board size 27 x 26.7 mm -> 28.9 x 26.7 mm
